File: StopWatchSender/StopWatchSender.sch (KiCad schematic (older format))
At the start: 3 parts

Commit message: wip
Parts:
- removed J?: Barrel_Jack, symbol Barrel_Jack
- added C1: CP, symbol CP
- added D1: LED, symbol LED
- added R1: 220, symbol R
- M-1: renamed from IC?; value ArduinoProMini -> ArduinoProMini 3.3V - 8MHZ
- gave numbers to parts that had none: 1
Connections:
- net GND: now also M-1.23 (GND), M-1.29 (GND), C1.2, D1.1 (K)
- net PB-Start3: now reaches M-1.10 ((PCINT23/AIN1)PD7/7)
- net at M-1.11 ((PCINT0/CLKO/ICP1)PB0/8): now also R1.2
- net at M-1.21 (VCC), M-2.2 (VCC): now also C1.1
- net VCC: now reaches M-1.24 (RAW)
- net PB-Stop: now reaches M-1.6 ((PCINT19/OC2B/INT1/PWM)PD3/3)
- net PB-Start0: now reaches M-1.7 ((PCINT20/XCK/T0)PD4/4)
- net PB-Start1: now reaches M-1.8 ((PCINT21/OC0B/T1/PWM)PD5/5)
- net PB-Start2: now reaches M-1.9 ((PCINT22/OC0A/AIN0/PWM)PD6/6)
- new net: D1.2 (A), R1.1
- no-connect marks 0 -> 11
Changed lines of the file:
@@
 LIBS:mysensors_arduino
 LIBS:mysensors_radios
+LIBS:StopWatchSender-cache
 EELAYER 25 0
 EELAYER END
@@
 encoding utf-8
 Sheet 1 1
-Title ""
-Date ""
+Title "StopWatch Sender"
+Date "2018-04-18"
 Rev ""
-Comp ""
-Comment1 ""
+Comp "G.S."
+Comment1 "ver. 0.1"
 Comment2 ""
 Comment3 ""
@@
 $EndDescr
 $Comp
-L ArduinoProMini IC?
+L ArduinoProMini M-1
 U 1 1 5AD6FFE1
 P 3800 2450
-F 0 "IC?" H 3050 3700 40  0000 L BNN
-F 1 "ArduinoProMini" H 4200 1050 40  0000 L BNN
+F 0 "M-1" H 3050 3700 40  0000 L BNN
+F 1 "ArduinoProMini 3.3V - 8MHZ" H 3750 1050 40  0000 L BNN
 F 2 "mysensors_arduino:pro_mini_china" H 3800 2450 30  0001 C CIN
 F 3 "" H 3800 2450 60  0000 C CNN
@@
 $EndComp
 $Comp
-L NRF24L01 U?
+L NRF24L01 M-2
 U 1 1 5AD70163
 P 6600 2400
-F 0 "U?" H 6700 2650 60  0000 C CNN
-F 1 "NRF24L01" H 6850 2150 60  0000 C CNN
+F 0 "M-2" H 6700 2650 60  0000 C CNN
+F 1 "NRF24L01" H 6250 2100 60  0000 C CNN
 F 2 "" H 6600 2250 60  0000 C CNN
 F 3 "" H 6600 2250 60  0000 C CNN
@@
 $EndComp
 $Comp
-L GND #PWR?
+L GND #PWR01
 U 1 1 5AD702E3
 P 6600 2750
-F 0 "#PWR?" H 6600 2500 50  0001 C CNN
+F 0 "#PWR01" H 6600 2500 50  0001 C CNN
 F 1 "GND" H 6600 2600 50  0000 C CNN
 F 2 "" H 6600 2750 50  0001 C CNN
@@
 $EndComp
 $Comp
-L Barrel_Jack J?
-U 1 1 5AD712E8
-P 1800 1750
-F 0 "J?" H 1800 1960 50  0000 C CNN
-F 1 "Barrel_Jack" H 1800 1575 50  0000 C CNN
-F 2 "" H 1850 1710 50  0001 C CNN
-F 3 "" H 1850 1710 50  0001 C CNN
-	1    1800 1750
-	1    0    0    -1
-$EndComp
-Wire Wire Line
-	4800 2650 5650 2650
-Wire Wire Line
-	5650 2650 5650 2300
-Wire Wire Line
-	5650 2300 6200 2300
-Wire Wire Line
-	4800 2550 5800 2550
-Wire Wire Line
-	5800 2550 5800 2400
-Wire Wire Line
-	5800 2400 6200 2400
-Wire Wire Line
-	4800 2750 5950 2750
-Wire Wire Line
-	5950 2750 5950 2500
-Wire Wire Line
-	5950 2500 6200 2500
-Wire Wire Line
-	4800 1550 7300 1550
-Wire Wire Line
-	7300 1550 7300 2400
-Wire Wire Line
-	7300 2400 7000 2400
-Wire Wire Line
-	4800 2250 5250 2250
-Wire Wire Line
-	5250 2250 5250 3100
-Wire Wire Line
-	7000 3100 7000 2500
-Wire Wire Line
-	4800 2350 5450 2350
-Wire Wire Line
-	5450 2350 5450 1750
-Wire Wire Line
-	5450 1750 7000 1750
-Wire Wire Line
-	7000 1750 7000 2300
-Wire Wire Line
-	5250 3100 7000 3100
-Wire Wire Line
-	2900 1350 2900 1000
-Wire Wire Line
-	2900 1000 6600 1000
-Wire Wire Line
-	6600 1000 6600 2050
-Wire Wire Line
-	2100 1650 2900 1650
-Wire Wire Line
-	2100 1850 2100 3900
-Wire Wire Line
-	2100 3450 2900 3450
-$Comp
-L GND #PWR?
+L GND #PWR02
 U 1 1 5AD717D9
 P 2100 3900
-F 0 "#PWR?" H 2100 3650 50  0001 C CNN
+F 0 "#PWR02" H 2100 3650 50  0001 C CNN
 F 1 "GND" H 2100 3750 50  0000 C CNN
 F 2 "" H 2100 3900 50  0001 C CNN
@@
 	1    0    0    -1
 $EndComp
-Connection ~ 2100 3450
+$Comp
+L LED D1
+U 1 1 5AD74996
+P 6600 3400
+F 0 "D1" H 6600 3500 50  0000 C CNN
+F 1 "LED" H 6600 3300 50  0000 C CNN
+F 2 "" H 6600 3400 50  0001 C CNN
+F 3 "" H 6600 3400 50  0001 C CNN
+	1    6600 3400
+	0    -1   -1   0
+$EndComp
+$Comp
+L GND #PWR03
+U 1 1 5AD74D48
+P 6600 3550
+F 0 "#PWR03" H 6600 3300 50  0001 C CNN
+F 1 "GND" H 6600 3400 50  0000 C CNN
+F 2 "" H 6600 3550 50  0001 C CNN
+F 3 "" H 6600 3550 50  0001 C CNN
+	1    6600 3550
+	1    0    0    -1
+$EndComp
+$Comp
+L R R1
+U 1 1 5AD74D78
+P 6100 3250
+F 0 "R1" V 6180 3250 50  0000 C CNN
+F 1 "220" V 6100 3250 50  0000 C CNN
+F 2 "" V 6030 3250 50  0001 C CNN
+F 3 "" H 6100 3250 50  0001 C CNN
+	1    6100 3250
+	0    1    1    0
+$EndComp
+$Comp
+L CP C1
+U 1 1 5AD752D4
+P 6150 2000
+F 0 "C1" H 6175 2100 50  0000 L CNN
+F 1 "CP" H 6175 1900 50  0000 L CNN
+F 2 "" H 6188 1850 50  0001 C CNN
+F 3 "" H 6150 2000 50  0001 C CNN
+	1    6150 2000
+	0    1    1    0
+$EndComp
+$Comp
+L GND #PWR04
+U 1 1 5AD7541E
+P 6000 2000
+F 0 "#PWR04" H 6000 1750 50  0001 C CNN
+F 1 "GND" H 6000 1850 50  0000 C CNN
+F 2 "" H 6000 2000 50  0001 C CNN
+F 3 "" H 6000 2000 50  0001 C CNN
+	1    6000 2000
+	1    0    0    -1
+$EndComp
+NoConn ~ 2900 3150
+NoConn ~ 2900 3250
+NoConn ~ 4800 3050
+NoConn ~ 4800 3150
+NoConn ~ 4800 3250
+NoConn ~ 4800 3350
+NoConn ~ 4800 3450
+NoConn ~ 4800 3550
+NoConn ~ 4800 3650
+NoConn ~ 4800 1350
+NoConn ~ 4800 1450
+Text GLabel 4800 1650 2    60   Input ~ 0
+PB-Stop
+Text GLabel 4800 1750 2    60   Input ~ 0
+PB-Start0
+Text GLabel 4800 1850 2    60   Input ~ 0
+PB-Start1
+Text GLabel 4800 1950 2    60   Input ~ 0
+PB-Start2
+Text GLabel 4800 2050 2    60   Input ~ 0
+PB-Start3
+Wire Wire Line
+	4800 2650 5650 2650
+Wire Wire Line
+	5650 2650 5650 2300
+Wire Wire Line
+	5650 2300 6200 2300
+Wire Wire Line
+	4800 2550 5800 2550
+Wire Wire Line
+	5800 2550 5800 2400
+Wire Wire Line
+	5800 2400 6200 2400
+Wire Wire Line
+	4800 2750 5950 2750
+Wire Wire Line
+	5950 2750 5950 2500
+Wire Wire Line
+	5950 2500 6200 2500
+Wire Wire Line
+	4800 1550 7300 1550
+Wire Wire Line
+	7300 1550 7300 2400
+Wire Wire Line
+	7300 2400 7000 2400
+Wire Wire Line
+	4800 2250 5250 2250
+Wire Wire Line
+	5250 2250 5250 3100
+Wire Wire Line
+	7000 3100 7000 2500
+Wire Wire Line
+	4800 2350 5450 2350
+Wire Wire Line
+	5450 2350 5450 1750
+Wire Wire Line
+	5450 1750 7000 1750
+Wire Wire Line
+	7000 1750 7000 2300
+Wire Wire Line
+	5250 3100 7000 3100
+Wire Wire Line
+	2900 1350 2900 1000
+Wire Wire Line
+	2900 1000 6600 1000
+Wire Wire Line
+	6600 1000 6600 2050
+Wire Wire Line
+	2100 1650 2900 1650
+Wire Wire Line
+	6250 3250 6600 3250
+Wire Wire Line
+	5950 3250 5050 3250
+Wire Wire Line
+	5050 3250 5050 2150
+Wire Wire Line
+	5050 2150 4800 2150
+Wire Wire Line
+	6300 2000 6600 2000
+Connection ~ 6600 2000
+Wire Wire Line
+	2900 3450 2900 3650
+Connection ~ 2900 3550
+Connection ~ 2900 3450
+Wire Wire Line
+	2100 3900 2100 3550
+Wire Wire Line
+	2100 3550 2900 3550
+$Comp
+L VCC #PWR05
+U 1 1 5AD76D94
+P 2100 1650
+F 0 "#PWR05" H 2100 1500 50  0001 C CNN
+F 1 "VCC" H 2100 1800 50  0000 C CNN
+F 2 "" H 2100 1650 50  0001 C CNN
+F 3 "" H 2100 1650 50  0001 C CNN
+	1    2100 1650
+	1    0    0    -1
+$EndComp
+$Comp
+L PWR_FLAG #FLG06
+U 1 1 5AD76E4A
+P 950 1000
+F 0 "#FLG06" H 950 1075 50  0001 C CNN
+F 1 "PWR_FLAG" H 950 1150 50  0000 C CNN
+F 2 "" H 950 1000 50  0001 C CNN
+F 3 "" H 950 1000 50  0001 C CNN
+	1    950  1000
+	1    0    0    -1
+$EndComp
+$Comp
+L PWR_FLAG #FLG07
+U 1 1 5AD76E68
+P 1550 1000
+F 0 "#FLG07" H 1550 1075 50  0001 C CNN
+F 1 "PWR_FLAG" H 1550 1150 50  0000 C CNN
+F 2 "" H 1550 1000 50  0001 C CNN
+F 3 "" H 1550 1000 50  0001 C CNN
+	1    1550 1000
+	1    0    0    -1
+$EndComp
+$Comp
+L GND #PWR08
+U 1 1 5AD76F0F
+P 1550 1000
+F 0 "#PWR08" H 1550 750 50  0001 C CNN
+F 1 "GND" H 1550 850 50  0000 C CNN
+F 2 "" H 1550 1000 50  0001 C CNN
+F 3 "" H 1550 1000 50  0001 C CNN
+	1    1550 1000
+	1    0    0    -1
+$EndComp
+$Comp
+L VCC #PWR09
+U 1 1 5AD76F2D
+P 950 1000
+F 0 "#PWR09" H 950 850 50  0001 C CNN
+F 1 "VCC" H 950 1150 50  0000 C CNN
+F 2 "" H 950 1000 50  0001 C CNN
+F 3 "" H 950 1000 50  0001 C CNN
+	1    950  1000
+	-1   0    0    1
+$EndComp
+Text GLabel 5200 2950 0    60   Output ~ 0
+AmpOut
 $EndSCHEMATC

Commit message: KiCad PCB update
Parts:
- removed M-1: ArduinoProMini 3.3V - 8MHZ, mysensors_arduino:pro_mini_china, symbol ArduinoProMini
- removed M-2: NRF24L01, symbol NRF24L01
- added IC1: ArduinoProMini, mysensors_arduino:pro_mini_china, symbol ArduinoProMini
- added J1: Conn_01x02_Male, symbol Conn_01x02_Male
- added SW1, SW2, SW3, SW4, SW5: SW_SPST, symbol SW_SPST
- added U1: NRF24L01, symbol NRF24L01
- R1: value 220 -> R
Connections:
- net GND: now also IC1.23 (GND), IC1.29 (GND), IC1.4 (GND), J1.1 (Pin_1), SW1.1 (A), SW2.1 (A), SW3.1 (A), SW4.1 (A), SW5.1 (A), U1.1 (GND)
- net at R1.2: now also D1.2 (A)
- net 3.3V: now reaches C1.1
- net 3.3V: now also IC1.21 (VCC), U1.2 (VCC)
- net R_LedClick: now reaches R1.1
- net R_LedClick: now also IC1.11 ((PCINT0/CLKO/ICP1)PB0/8); no longer D1.2 (A)
- new net +5V: IC1.24 (RAW)
- new net Click_Amp: IC1.17 ((PCINT8/ADC0)PC0/14/A0), J1.2 (Pin_2)
- new net PB_Start0: IC1.7 ((PCINT20/XCK/T0)PD4/4), SW2.2 (B)
- new net PB_Start1: IC1.8 ((PCINT21/OC0B/T1/PWM)PD5/5), SW3.2 (B)
- new net PB_Start2: IC1.9 ((PCINT22/OC0A/AIN0/PWM)PD6/6), SW4.2 (B)
- new net PB_Start3: IC1.10 ((PCINT23/AIN1)PD7/7), SW5.2 (B)
- new net PB_Stop: IC1.6 ((PCINT19/OC2B/INT1/PWM)PD3/3), SW1.2 (B)
- new net nRF_CE: IC1.12 ((PCINT1/OC1A/PWM)PB1/9), U1.3 (CE)
- new net nRF_CSN: IC1.13 ((PCINT2/OC1B/~SS~/PWM)PB2/10), U1.4 (CSN)
- new net nRF_IRQ: IC1.5 ((PCINT18/INT0)PD2/2), U1.8 (IRQ)
- new net nRF_MISO: IC1.15 ((PCINT4/MISO)PB4/12), U1.7 (MISO)
- new net nRF_MOSI: IC1.14 ((PCINT3/OC2A/MOSI/PWM)PB3/11), U1.6 (MOSI)
- new net nRF_SCK: IC1.16 ((PCINT5/SCK)PB5/13), U1.5 (SCK)

Commit message: KiCad PCB update
Parts:
- C1: footprint (none) -> Capacitors_THT:CP_Radial_D4.0mm_P1.50mm
- IC1: footprint mysensors_arduino:pro_mini_china -> mysensors_arduino:pro_mini
- U1: footprint (none) -> mysensors_radios:NRF24L01
Changed lines of the file:
@@
 F 0 "IC1" H 1750 3750 40  0000 L BNN
 F 1 "ArduinoProMini" H 2900 1100 40  0000 L BNN
-F 2 "mysensors_arduino:pro_mini_china" H 2500 2500 30  0001 C CIN
+F 2 "mysensors_arduino:pro_mini" H 2500 2500 30  0001 C CIN
 F 3 "" H 2500 2500 60  0000 C CNN
 	1    2500 2500
@@
 F 0 "U1" H 7350 2950 60  0000 C CNN
 F 1 "NRF24L01" H 7500 2450 60  0000 C CNN
-F 2 "" H 7250 2550 60  0000 C CNN
+F 2 "mysensors_radios:NRF24L01" H 7250 2550 60  0000 C CNN
 F 3 "" H 7250 2550 60  0000 C CNN
 	1    7250 2700
@@
 F 0 "C1" H 7275 2100 50  0000 L CNN
 F 1 "CP" H 7275 1900 50  0000 L CNN
-F 2 "" H 7288 1850 50  0001 C CNN
+F 2 "Capacitors_THT:CP_Radial_D4.0mm_P1.50mm" H 7288 1850 50  0001 C CNN
 F 3 "" H 7250 2000 50  0001 C CNN
 	1    7250 2000

Commit message: Working on the electronics
Parts:
- removed SW1, SW2, SW3, SW4, SW5: SW_SPST, symbol SW_SPST
- added J2: Conn_01x06, Pin_Headers:Pin_Header_Straight_1x06_Pitch2.54mm, symbol Conn_01x06
- D1: footprint (none) -> LEDs:LED_D4.0mm
- J1: footprint (none) -> Pin_Headers:Pin_Header_Straight_1x02_Pitch2.54mm
- R1: footprint (none) -> Resistors_THT:R_Axial_DIN0207_L6.3mm_D2.5mm_P10.16mm_Horizontal
Connections:
- net GND: now also J2.6 (Pin_6)
- net PB_Start0: now also J2.4 (Pin_4)
- net PB_Start1: now also J2.3 (Pin_3)
- net PB_Start2: now also J2.2 (Pin_2)
- net PB_Start3: now also J2.1 (Pin_1)
- net PB_Stop: now also J2.5 (Pin_5)
- no-connect marks 11 -> 12
Changed lines of the file:
@@
 $EndDescr
-$Comp
-L ArduinoProMini IC1
-U 1 1 5AD8A133
-P 2500 2500
-F 0 "IC1" H 1750 3750 40  0000 L BNN
-F 1 "ArduinoProMini" H 2900 1100 40  0000 L BNN
-F 2 "mysensors_arduino:pro_mini" H 2500 2500 30  0001 C CIN
-F 3 "" H 2500 2500 60  0000 C CNN
-	1    2500 2500
-	1    0    0    -1
-$EndComp
 $Comp
 L NRF24L01 U1
@@
 F 0 "D1" H 4900 4350 50  0000 C CNN
 F 1 "LED" H 4900 4150 50  0000 C CNN
-F 2 "" H 4900 4250 50  0001 C CNN
+F 2 "LEDs:LED_D4.0mm" H 4900 4250 50  0001 C CNN
 F 3 "" H 4900 4250 50  0001 C CNN
 	1    4900 4250
@@
 F 0 "R1" V 4980 3950 50  0000 C CNN
 F 1 "R" V 4900 3950 50  0000 C CNN
-F 2 "" V 4830 3950 50  0001 C CNN
+F 2 "Resistors_THT:R_Axial_DIN0207_L6.3mm_D2.5mm_P10.16mm_Horizontal" V 4830 3950 50  0001 C CNN
 F 3 "" H 4900 3950 50  0001 C CNN
 	1    4900 3950
@@
 	1    7250 2000
 	-1   0    0    1
-$EndComp
-$Comp
-L SW_SPST SW1
-U 1 1 5AD8A6FC
-P 6100 4600
-F 0 "SW1" H 6100 4725 50  0000 C CNN
-F 1 "SW_SPST" H 6100 4500 50  0000 C CNN
-F 2 "" H 6100 4600 50  0001 C CNN
-F 3 "" H 6100 4600 50  0001 C CNN
-	1    6100 4600
-	0    -1   -1   0
-$EndComp
-$Comp
-L SW_SPST SW2
-U 1 1 5AD8A828
-P 6550 4600
-F 0 "SW2" H 6550 4725 50  0000 C CNN
-F 1 "SW_SPST" H 6550 4500 50  0000 C CNN
-F 2 "" H 6550 4600 50  0001 C CNN
-F 3 "" H 6550 4600 50  0001 C CNN
-	1    6550 4600
-	0    -1   -1   0
-$EndComp
-$Comp
-L SW_SPST SW3
-U 1 1 5AD8A86D
-P 7000 4600
-F 0 "SW3" H 7000 4725 50  0000 C CNN
-F 1 "SW_SPST" H 7000 4500 50  0000 C CNN
-F 2 "" H 7000 4600 50  0001 C CNN
-F 3 "" H 7000 4600 50  0001 C CNN
-	1    7000 4600
-	0    -1   -1   0
-$EndComp
-$Comp
-L SW_SPST SW4
-U 1 1 5AD8A8CA
-P 7450 4600
-F 0 "SW4" H 7450 4725 50  0000 C CNN
-F 1 "SW_SPST" H 7450 4500 50  0000 C CNN
-F 2 "" H 7450 4600 50  0001 C CNN
-F 3 "" H 7450 4600 50  0001 C CNN
-	1    7450 4600
-	0    -1   -1   0
-$EndComp
-$Comp
-L SW_SPST SW5
-U 1 1 5AD8A913
-P 7900 4600
-F 0 "SW5" H 7900 4725 50  0000 C CNN
-F 1 "SW_SPST" H 7900 4500 50  0000 C CNN
-F 2 "" H 7900 4600 50  0001 C CNN
-F 3 "" H 7900 4600 50  0001 C CNN
-	1    7900 4600
-	0    -1   -1   0
 $EndComp
 $Comp
@@
 	1    0    0    -1
 $EndComp
-$Comp
-L GND #PWR03
-U 1 1 5AD8C1F6
-P 6100 4800
-F 0 "#PWR03" H 6100 4550 50  0001 C CNN
-F 1 "GND" H 6100 4650 50  0000 C CNN
-F 2 "" H 6100 4800 50  0001 C CNN
-F 3 "" H 6100 4800 50  0001 C CNN
-	1    6100 4800
-	1    0    0    -1
-$EndComp
+Wire Wire Line
+	7250 2350 7250 2150
 $Comp
 L GND #PWR04
-U 1 1 5AD8C251
-P 6550 4800
-F 0 "#PWR04" H 6550 4550 50  0001 C CNN
-F 1 "GND" H 6550 4650 50  0000 C CNN
-F 2 "" H 6550 4800 50  0001 C CNN
-F 3 "" H 6550 4800 50  0001 C CNN
-	1    6550 4800
-	1    0    0    -1
-$EndComp
-$Comp
-L GND #PWR05
-U 1 1 5AD8C27A
-P 7000 4800
-F 0 "#PWR05" H 7000 4550 50  0001 C CNN
-F 1 "GND" H 7000 4650 50  0000 C CNN
-F 2 "" H 7000 4800 50  0001 C CNN
-F 3 "" H 7000 4800 50  0001 C CNN
-	1    7000 4800
-	1    0    0    -1
-$EndComp
-$Comp
-L GND #PWR06
-U 1 1 5AD8C2A3
-P 7450 4800
-F 0 "#PWR06" H 7450 4550 50  0001 C CNN
-F 1 "GND" H 7450 4650 50  0000 C CNN
-F 2 "" H 7450 4800 50  0001 C CNN
-F 3 "" H 7450 4800 50  0001 C CNN
-	1    7450 4800
-	1    0    0    -1
-$EndComp
-$Comp
-L GND #PWR07
-U 1 1 5AD8C678
-P 7900 4800
-F 0 "#PWR07" H 7900 4550 50  0001 C CNN
-F 1 "GND" H 7900 4650 50  0000 C CNN
-F 2 "" H 7900 4800 50  0001 C CNN
-F 3 "" H 7900 4800 50  0001 C CNN
-	1    7900 4800
-	1    0    0    -1
-$EndComp
-$Comp
-L GND #PWR08
-U 1 1 5AD8C6A1
-P 1600 3700
-F 0 "#PWR08" H 1600 3450 50  0001 C CNN
-F 1 "GND" H 1600 3550 50  0000 C CNN
-F 2 "" H 1600 3700 50  0001 C CNN
-F 3 "" H 1600 3700 50  0001 C CNN
-	1    1600 3700
-	1    0    0    -1
-$EndComp
-Wire Wire Line
-	1600 3500 1600 3700
-Connection ~ 1600 3600
-Wire Wire Line
-	7250 2350 7250 2150
-$Comp
-L GND #PWR09
 U 1 1 5AD8C98E
 P 7650 1850
-F 0 "#PWR09" H 7650 1600 50  0001 C CNN
+F 0 "#PWR04" H 7650 1600 50  0001 C CNN
 F 1 "GND" H 7650 1700 50  0000 C CNN
 F 2 "" H 7650 1850 50  0001 C CNN
@@
 Wire Wire Line
 	7250 1850 7650 1850
-Text Label 6100 4400 1    60   ~ 0
-PB_Stop
 Text Label 3500 1700 0    60   ~ 0
 PB_Stop
-Text Label 6550 4400 1    60   ~ 0
-PB_Start0
 Text Label 3500 1800 0    60   ~ 0
 PB_Start0
 Text Label 3500 1900 0    60   ~ 0
 PB_Start1
-Text Label 7000 4400 1    60   ~ 0
-PB_Start1
-Text Label 7450 4400 1    60   ~ 0
-PB_Start2
 Text Label 3500 2000 0    60   ~ 0
 PB_Start2
 Text Label 3500 2100 0    60   ~ 0
-PB_Start3
-Text Label 7900 4400 1    60   ~ 0
 PB_Start3
 NoConn ~ 1600 3200
@@
 R_LedClick
 $Comp
-L GND #PWR010
+L GND #PWR05
 U 1 1 5AD8D2F2
 P 4900 4400
-F 0 "#PWR010" H 4900 4150 50  0001 C CNN
+F 0 "#PWR05" H 4900 4150 50  0001 C CNN
 F 1 "GND" H 4900 4250 50  0000 C CNN
 F 2 "" H 4900 4400 50  0001 C CNN
@@
 F 0 "J1" H 4100 4150 50  0000 C CNN
 F 1 "Conn_01x02_Male" H 4100 3850 50  0000 C CNN
-F 2 "" H 4100 4050 50  0001 C CNN
+F 2 "Pin_Headers:Pin_Header_Straight_1x02_Pitch2.54mm" H 4100 4050 50  0001 C CNN
 F 3 "" H 4100 4050 50  0001 C CNN
 	1    4100 4050
@@
 $EndComp
 $Comp
-L GND #PWR011
+L GND #PWR06
 U 1 1 5AD8D652
 P 4100 4250
-F 0 "#PWR011" H 4100 4000 50  0001 C CNN
+F 0 "#PWR06" H 4100 4000 50  0001 C CNN
 F 1 "GND" H 4100 4100 50  0000 C CNN
 F 2 "" H 4100 4250 50  0001 C CNN
@@
 Click_Amp
 $Comp
-L PWR_FLAG #FLG012
+L PWR_FLAG #FLG07
 U 1 1 5AD8D983
 P 5300 800
-F 0 "#FLG012" H 5300 875 50  0001 C CNN
+F 0 "#FLG07" H 5300 875 50  0001 C CNN
 F 1 "PWR_FLAG" H 5300 950 50  0000 C CNN
 F 2 "" H 5300 800 50  0001 C CNN
@@
 $EndComp
 $Comp
-L PWR_FLAG #FLG013
+L PWR_FLAG #FLG08
 U 1 1 5AD8D9B6
 P 5750 800
-F 0 "#FLG013" H 5750 875 50  0001 C CNN
+F 0 "#FLG08" H 5750 875 50  0001 C CNN
 F 1 "PWR_FLAG" H 5750 950 50  0000 C CNN
 F 2 "" H 5750 800 50  0001 C CNN
@@
 $EndComp
 $Comp
-L GND #PWR014
+L GND #PWR09
 U 1 1 5AD8DA5D
 P 5750 800
-F 0 "#PWR014" H 5750 550 50  0001 C CNN
+F 0 "#PWR09" H 5750 550 50  0001 C CNN
 F 1 "GND" H 5750 650 50  0000 C CNN
 F 2 "" H 5750 800 50  0001 C CNN
@@
 $EndComp
 $Comp
-L +5V #PWR015
+L +5V #PWR010
 U 1 1 5AD8DDA9
 P 5300 800
-F 0 "#PWR015" H 5300 650 50  0001 C CNN
+F 0 "#PWR010" H 5300 650 50  0001 C CNN
 F 1 "+5V" H 5300 940 50  0000 C CNN
 F 2 "" H 5300 800 50  0001 C CNN
@@
 NoConn ~ 3500 1400
 NoConn ~ 3500 1500
+$Comp
+L Conn_01x06 J2
+U 1 1 5AD9B7F7
+P 6000 3550
+F 0 "J2" H 6000 3850 50  0000 C CNN
+F 1 "Conn_01x06" H 6000 3150 50  0000 C CNN
+F 2 "Pin_Headers:Pin_Header_Straight_1x06_Pitch2.54mm" H 6000 3550 50  0001 C CNN
+F 3 "" H 6000 3550 50  0001 C CNN
+	1    6000 3550
+	0    1    1    0
+$EndComp
+Text Label 5800 3350 1    60   ~ 0
+PB_Stop
+Text Label 5900 3350 1    60   ~ 0
+PB_Start0
+Text Label 6000 3350 1    60   ~ 0
+PB_Start1
+Text Label 6100 3350 1    60   ~ 0
+PB_Start2
+Text Label 6200 3350 1    60   ~ 0
+PB_Start3
+$Comp
+L GND #PWR011
+U 1 1 5AD9B9F1
+P 5400 3550
+F 0 "#PWR011" H 5400 3300 50  0001 C CNN
+F 1 "GND" H 5400 3400 50  0000 C CNN
+F 2 "" H 5400 3550 50  0001 C CNN
+F 3 "" H 5400 3550 50  0001 C CNN
+	1    5400 3550
+	1    0    0    -1
+$EndComp
+Wire Wire Line
+	5700 3350 5400 3350
+Wire Wire Line
+	5400 3350 5400 3550
+$Comp
+L ArduinoProMini IC1
+U 1 1 5AD8A133
+P 2500 2500
+F 0 "IC1" H 1750 3750 40  0000 L BNN
+F 1 "ArduinoProMini" H 2900 1100 40  0000 L BNN
+F 2 "mysensors_arduino:pro_mini" H 2500 2500 30  0001 C CIN
+F 3 "" H 2500 2500 60  0000 C CNN
+	1    2500 2500
+	1    0    0    -1
+$EndComp
+NoConn ~ 2050 -400
+$Comp
+L GND #PWR?
+U 1 1 5AD9C43E
+P 1050 3700
+F 0 "#PWR?" H 1050 3450 50  0001 C CNN
+F 1 "GND" H 1050 3550 50  0000 C CNN
+F 2 "" H 1050 3700 50  0001 C CNN
+F 3 "" H 1050 3700 50  0001 C CNN
+	1    1050 3700
+	1    0    0    -1
+$EndComp
+$Comp
+L GND #PWR?
+U 1 1 5AD9C41E
+P 1350 3700
+F 0 "#PWR?" H 1350 3450 50  0001 C CNN
+F 1 "GND" H 1350 3550 50  0000 C CNN
+F 2 "" H 1350 3700 50  0001 C CNN
+F 3 "" H 1350 3700 50  0001 C CNN
+	1    1350 3700
+	1    0    0    -1
+$EndComp
+$Comp
+L GND #PWR03
+U 1 1 5AD8C6A1
+P 1600 3700
+F 0 "#PWR03" H 1600 3450 50  0001 C CNN
+F 1 "GND" H 1600 3550 50  0000 C CNN
+F 2 "" H 1600 3700 50  0001 C CNN
+F 3 "" H 1600 3700 50  0001 C CNN
+	1    1600 3700
+	1    0    0    -1
+$EndComp
+Wire Wire Line
+	1600 3600 1350 3600
+Wire Wire Line
+	1350 3600 1350 3700
+Wire Wire Line
+	1600 3500 1050 3500
+Wire Wire Line
+	1050 3500 1050 3700
 $EndSCHEMATC
