File: StopWatchSender/StopWatchSender.sch (KiCad schematic (older format))
At the start: 7 parts, among them IC1 ArduinoProMini, J1 Conn_01x02_Male, J2 Conn_01x06, U1 NRF24L01

Commit message: wip
Parts:
- removed J2: Conn_01x06, Pin_Headers:Pin_Header_Straight_1x06_Pitch2.54mm, symbol Conn_01x06
- added J2: Barrel_Jack, mysensors_connectors:dc_socket-kcswalter, symbol Barrel_Jack
- added SW1, SW2, SW3, SW4, SW5: SW_Push, Buttons_Switches_THT:SW_PUSH_6mm_h8mm, symbol SW_Push
- U1: footprint mysensors_radios:NRF24L01 -> mysensors_radios:NRF24L01_PA_LNA-SMD
Connections:
- net +5V: now also J2.1
- net GND: now also J2.2, SW1.2, SW2.2, SW3.2, SW4.2, SW5.2
- net PB_Start0: now also SW2.1
- net PB_Start1: now also SW3.1
- net PB_Start2: now also SW4.1
- net PB_Start3: now also SW5.1
- net PB_Stop: now also SW1.1
Changed lines of the file:
@@
 F 0 "U1" H 7350 2950 60  0000 C CNN
 F 1 "NRF24L01" H 7500 2450 60  0000 C CNN
-F 2 "mysensors_radios:NRF24L01" H 7250 2550 60  0000 C CNN
+F 2 "mysensors_radios:NRF24L01_PA_LNA-SMD" H 5900 3100 60  0000 C CNN
 F 3 "" H 7250 2550 60  0000 C CNN
 	1    7250 2700
@@
 $EndComp
 $Comp
-L +5V #PWR01
+L +5V #PWR1
 U 1 1 5AD8AA5B
 P 1200 1050
-F 0 "#PWR01" H 1200 900 50  0001 C CNN
+F 0 "#PWR1" H 1200 900 50  0001 C CNN
 F 1 "+5V" H 1200 1190 50  0000 C CNN
 F 2 "" H 1200 1050 50  0001 C CNN
@@
 	1    0    0    -1
 $EndComp
-Wire Wire Line
-	1200 1050 1200 1700
-Wire Wire Line
-	1200 1700 1600 1700
 Text Label 3500 1600 0    60   ~ 0
 nRF_IRQ
@@
 3.3V
 $Comp
-L GND #PWR02
+L GND #PWR10
 U 1 1 5AD8C1C6
 P 7250 3050
-F 0 "#PWR02" H 7250 2800 50  0001 C CNN
+F 0 "#PWR10" H 7250 2800 50  0001 C CNN
 F 1 "GND" H 7250 2900 50  0000 C CNN
 F 2 "" H 7250 3050 50  0001 C CNN
@@
 	1    0    0    -1
 $EndComp
-Wire Wire Line
-	7250 2350 7250 2150
-$Comp
-L GND #PWR04
+$Comp
+L GND #PWR12
 U 1 1 5AD8C98E
 P 7650 1850
-F 0 "#PWR04" H 7650 1600 50  0001 C CNN
+F 0 "#PWR12" H 7650 1600 50  0001 C CNN
 F 1 "GND" H 7650 1700 50  0000 C CNN
 F 2 "" H 7650 1850 50  0001 C CNN
@@
 	1    0    0    -1
 $EndComp
-Wire Wire Line
-	7250 1850 7650 1850
 Text Label 3500 1700 0    60   ~ 0
 PB_Stop
@@
 R_LedClick
 $Comp
-L GND #PWR05
+L GND #PWR6
 U 1 1 5AD8D2F2
 P 4900 4400
-F 0 "#PWR05" H 4900 4150 50  0001 C CNN
+F 0 "#PWR6" H 4900 4150 50  0001 C CNN
 F 1 "GND" H 4900 4250 50  0000 C CNN
 F 2 "" H 4900 4400 50  0001 C CNN
@@
 $EndComp
 $Comp
-L GND #PWR06
+L GND #PWR5
 U 1 1 5AD8D652
 P 4100 4250
-F 0 "#PWR06" H 4100 4000 50  0001 C CNN
+F 0 "#PWR5" H 4100 4000 50  0001 C CNN
 F 1 "GND" H 4100 4100 50  0000 C CNN
 F 2 "" H 4100 4250 50  0001 C CNN
@@
 Click_Amp
 $Comp
-L PWR_FLAG #FLG07
+L PWR_FLAG #FLG1
 U 1 1 5AD8D983
 P 5300 800
-F 0 "#FLG07" H 5300 875 50  0001 C CNN
+F 0 "#FLG1" H 5300 875 50  0001 C CNN
 F 1 "PWR_FLAG" H 5300 950 50  0000 C CNN
 F 2 "" H 5300 800 50  0001 C CNN
@@
 $EndComp
 $Comp
-L PWR_FLAG #FLG08
+L PWR_FLAG #FLG2
 U 1 1 5AD8D9B6
 P 5750 800
-F 0 "#FLG08" H 5750 875 50  0001 C CNN
+F 0 "#FLG2" H 5750 875 50  0001 C CNN
 F 1 "PWR_FLAG" H 5750 950 50  0000 C CNN
 F 2 "" H 5750 800 50  0001 C CNN
@@
 $EndComp
 $Comp
-L GND #PWR09
+L GND #PWR8
 U 1 1 5AD8DA5D
 P 5750 800
-F 0 "#PWR09" H 5750 550 50  0001 C CNN
+F 0 "#PWR8" H 5750 550 50  0001 C CNN
 F 1 "GND" H 5750 650 50  0000 C CNN
 F 2 "" H 5750 800 50  0001 C CNN
@@
 $EndComp
 $Comp
-L +5V #PWR010
+L +5V #PWR7
 U 1 1 5AD8DDA9
 P 5300 800
-F 0 "#PWR010" H 5300 650 50  0001 C CNN
+F 0 "#PWR7" H 5300 650 50  0001 C CNN
 F 1 "+5V" H 5300 940 50  0000 C CNN
 F 2 "" H 5300 800 50  0001 C CNN
@@
 NoConn ~ 3500 1400
 NoConn ~ 3500 1500
-$Comp
-L Conn_01x06 J2
-U 1 1 5AD9B7F7
-P 6000 3550
-F 0 "J2" H 6000 3850 50  0000 C CNN
-F 1 "Conn_01x06" H 6000 3150 50  0000 C CNN
-F 2 "Pin_Headers:Pin_Header_Straight_1x06_Pitch2.54mm" H 6000 3550 50  0001 C CNN
-F 3 "" H 6000 3550 50  0001 C CNN
-	1    6000 3550
-	0    1    1    0
-$EndComp
-Text Label 5800 3350 1    60   ~ 0
-PB_Stop
-Text Label 5900 3350 1    60   ~ 0
-PB_Start0
-Text Label 6000 3350 1    60   ~ 0
-PB_Start1
-Text Label 6100 3350 1    60   ~ 0
-PB_Start2
-Text Label 6200 3350 1    60   ~ 0
-PB_Start3
-$Comp
-L GND #PWR011
-U 1 1 5AD9B9F1
-P 5400 3550
-F 0 "#PWR011" H 5400 3300 50  0001 C CNN
-F 1 "GND" H 5400 3400 50  0000 C CNN
-F 2 "" H 5400 3550 50  0001 C CNN
-F 3 "" H 5400 3550 50  0001 C CNN
-	1    5400 3550
-	1    0    0    -1
-$EndComp
-Wire Wire Line
-	5700 3350 5400 3350
-Wire Wire Line
-	5400 3350 5400 3550
 $Comp
 L ArduinoProMini IC1
@@
 NoConn ~ 2050 -400
 $Comp
-L GND #PWR?
-U 1 1 5AD9C43E
-P 1050 3700
-F 0 "#PWR?" H 1050 3450 50  0001 C CNN
-F 1 "GND" H 1050 3550 50  0000 C CNN
-F 2 "" H 1050 3700 50  0001 C CNN
-F 3 "" H 1050 3700 50  0001 C CNN
-	1    1050 3700
-	1    0    0    -1
-$EndComp
-$Comp
-L GND #PWR?
-U 1 1 5AD9C41E
-P 1350 3700
-F 0 "#PWR?" H 1350 3450 50  0001 C CNN
-F 1 "GND" H 1350 3550 50  0000 C CNN
-F 2 "" H 1350 3700 50  0001 C CNN
-F 3 "" H 1350 3700 50  0001 C CNN
-	1    1350 3700
-	1    0    0    -1
-$EndComp
-$Comp
-L GND #PWR03
-U 1 1 5AD8C6A1
+L GND #PWR2
+U 1 1 5ADD932B
 P 1600 3700
-F 0 "#PWR03" H 1600 3450 50  0001 C CNN
+F 0 "#PWR2" H 1600 3450 50  0001 C CNN
 F 1 "GND" H 1600 3550 50  0000 C CNN
 F 2 "" H 1600 3700 50  0001 C CNN
@@
 	1    0    0    -1
 $EndComp
-Wire Wire Line
-	1600 3600 1350 3600
-Wire Wire Line
-	1350 3600 1350 3700
-Wire Wire Line
-	1600 3500 1050 3500
-Wire Wire Line
-	1050 3500 1050 3700
+$Comp
+L SW_Push SW1
+U 1 1 5ADDB336
+P 6850 4200
+F 0 "SW1" H 6900 4300 50  0000 L CNN
+F 1 "SW_Push" H 6850 4140 50  0000 C CNN
+F 2 "Buttons_Switches_THT:SW_PUSH_6mm_h8mm" H 6850 4400 50  0001 C CNN
+F 3 "" H 6850 4400 50  0001 C CNN
+	1    6850 4200
+	0    1    1    0
+$EndComp
+$Comp
+L SW_Push SW2
+U 1 1 5ADDB3ED
+P 7300 4200
+F 0 "SW2" H 7350 4300 50  0000 L CNN
+F 1 "SW_Push" H 7300 4140 50  0000 C CNN
+F 2 "Buttons_Switches_THT:SW_PUSH_6mm_h8mm" H 7300 4400 50  0001 C CNN
+F 3 "" H 7300 4400 50  0001 C CNN
+	1    7300 4200
+	0    1    1    0
+$EndComp
+$Comp
+L SW_Push SW3
+U 1 1 5ADDB42E
+P 7750 4200
+F 0 "SW3" H 7800 4300 50  0000 L CNN
+F 1 "SW_Push" H 7750 4140 50  0000 C CNN
+F 2 "Buttons_Switches_THT:SW_PUSH_6mm_h8mm" H 7750 4400 50  0001 C CNN
+F 3 "" H 7750 4400 50  0001 C CNN
+	1    7750 4200
+	0    1    1    0
+$EndComp
+$Comp
+L SW_Push SW4
+U 1 1 5ADDB47C
+P 8200 4200
+F 0 "SW4" H 8250 4300 50  0000 L CNN
+F 1 "SW_Push" H 8200 4140 50  0000 C CNN
+F 2 "Buttons_Switches_THT:SW_PUSH_6mm_h8mm" H 8200 4400 50  0001 C CNN
+F 3 "" H 8200 4400 50  0001 C CNN
+	1    8200 4200
+	0    1    1    0
+$EndComp
+$Comp
+L SW_Push SW5
+U 1 1 5ADDB4BF
+P 8650 4200
+F 0 "SW5" H 8700 4300 50  0000 L CNN
+F 1 "SW_Push" H 8650 4140 50  0000 C CNN
+F 2 "Buttons_Switches_THT:SW_PUSH_6mm_h8mm" H 8650 4400 50  0001 C CNN
+F 3 "" H 8650 4400 50  0001 C CNN
+	1    8650 4200
+	0    1    1    0
+$EndComp
+$Comp
+L GND #PWR9
+U 1 1 5ADDB717
+P 6850 4400
+F 0 "#PWR9" H 6850 4150 50  0001 C CNN
+F 1 "GND" H 6850 4250 50  0000 C CNN
+F 2 "" H 6850 4400 50  0001 C CNN
+F 3 "" H 6850 4400 50  0001 C CNN
+	1    6850 4400
+	1    0    0    -1
+$EndComp
+$Comp
+L GND #PWR11
+U 1 1 5ADDB746
+P 7300 4400
+F 0 "#PWR11" H 7300 4150 50  0001 C CNN
+F 1 "GND" H 7300 4250 50  0000 C CNN
+F 2 "" H 7300 4400 50  0001 C CNN
+F 3 "" H 7300 4400 50  0001 C CNN
+	1    7300 4400
+	1    0    0    -1
+$EndComp
+$Comp
+L GND #PWR13
+U 1 1 5ADDB775
+P 7750 4400
+F 0 "#PWR13" H 7750 4150 50  0001 C CNN
+F 1 "GND" H 7750 4250 50  0000 C CNN
+F 2 "" H 7750 4400 50  0001 C CNN
+F 3 "" H 7750 4400 50  0001 C CNN
+	1    7750 4400
+	1    0    0    -1
+$EndComp
+$Comp
+L GND #PWR14
+U 1 1 5ADDB7A4
+P 8200 4400
+F 0 "#PWR14" H 8200 4150 50  0001 C CNN
+F 1 "GND" H 8200 4250 50  0000 C CNN
+F 2 "" H 8200 4400 50  0001 C CNN
+F 3 "" H 8200 4400 50  0001 C CNN
+	1    8200 4400
+	1    0    0    -1
+$EndComp
+$Comp
+L GND #PWR15
+U 1 1 5ADDB7D3
+P 8650 4400
+F 0 "#PWR15" H 8650 4150 50  0001 C CNN
+F 1 "GND" H 8650 4250 50  0000 C CNN
+F 2 "" H 8650 4400 50  0001 C CNN
+F 3 "" H 8650 4400 50  0001 C CNN
+	1    8650 4400
+	1    0    0    -1
+$EndComp
+Text Label 6850 4000 1    60   ~ 0
+PB_Stop
+Text Label 7300 4000 1    60   ~ 0
+PB_Start0
+Text Label 7750 4000 1    60   ~ 0
+PB_Start1
+Text Label 8200 4000 1    60   ~ 0
+PB_Start2
+Text Label 8650 4000 1    60   ~ 0
+PB_Start3
+Wire Wire Line
+	1200 1050 1200 1700
+Wire Wire Line
+	1200 1700 1600 1700
+Wire Wire Line
+	7250 2350 7250 2150
+Wire Wire Line
+	7250 1850 7650 1850
+Wire Wire Line
+	1600 3500 1600 3700
+Connection ~ 1600 3600
+$Comp
+L Barrel_Jack J2
+U 1 1 5ADDEC59
+P 2500 5950
+F 0 "J2" H 2500 6160 50  0000 C CNN
+F 1 "Barrel_Jack" H 2500 5775 50  0000 C CNN
+F 2 "mysensors_connectors:dc_socket-kcswalter" H 2550 5910 50  0001 C CNN
+F 3 "" H 2550 5910 50  0001 C CNN
+	1    2500 5950
+	1    0    0    -1
+$EndComp
+$Comp
+L GND #PWR4
+U 1 1 5ADDED47
+P 2800 6050
+F 0 "#PWR4" H 2800 5800 50  0001 C CNN
+F 1 "GND" H 2800 5900 50  0000 C CNN
+F 2 "" H 2800 6050 50  0001 C CNN
+F 3 "" H 2800 6050 50  0001 C CNN
+	1    2800 6050
+	1    0    0    -1
+$EndComp
+$Comp
+L +5V #PWR3
+U 1 1 5ADDEF4A
+P 2800 5850
+F 0 "#PWR3" H 2800 5700 50  0001 C CNN
+F 1 "+5V" H 2800 5990 50  0000 C CNN
+F 2 "" H 2800 5850 50  0001 C CNN
+F 3 "" H 2800 5850 50  0001 C CNN
+	1    2800 5850
+	1    0    0    -1
+$EndComp
 $EndSCHEMATC

Commit message: wip
Parts:
- added C2: 10nF, Capacitors_SMD:C_0603, symbol C
- added C3: 10pF, Capacitors_SMD:C_0603, symbol C
- added C4: C, Capacitors_SMD:C_0603, symbol C
- added C5: 100uF, Capacitors_THT:CP_Radial_D6.3mm_P2.50mm, symbol CP
- added D2: LED, LEDs:LED_0603, symbol LED
- added J3: Conn_01x04_Male, Pin_Headers:Pin_Header_Straight_1x04_Pitch2.54mm, symbol Conn_01x04_Male
- added J4: Screw_Terminal_01x02, mysensors_connectors:TerminalBlock2.54mmx2-kcswalter, symbol Screw_Terminal_01x02
- added R2: 1K, Resistors_SMD:R_0603, symbol R
- added R3: 0, Resistors_SMD:R_0603, symbol R
- added R4: 100, Resistors_SMD:R_0603, symbol R
- added RV1: 10K, Potentiometers:Potentiometer_Trimmer_ACP_CA6v_Horizontal, symbol POT
- added U2: LM386, SMD_Packages:SOIC-8-N, symbol LM386
- R1: footprint Resistors_THT:R_Axial_DIN0207_L6.3mm_D2.5mm_P10.16mm_Horizontal -> Resistors_THT:R_Axial_DIN0204_L3.6mm_D1.6mm_P5.08mm_Horizontal
- U1: footprint mysensors_radios:NRF24L01_PA_LNA-SMD -> mysensors_radios:NRF24L01
- renumbered J2 to J1, J1 to J2
Connections:
- wire segments 5 -> 18
- no-connect marks 12 -> 13
Other:
- moved on the sheet: C1, SW1, SW2, SW3, SW4, SW5, U1
