File: StopWatchSender/StopWatchSender.kicad_pcb (KiCad board)
At the start: 2 copper layers, 0 parts

Commit message: Working on the electronics
Parts:
- added C1: CP, Capacitors_THT:CP_Radial_D4.0mm_P1.50mm, F.Cu at (92.7, 73.7)
- added D1: LED, LEDs:LED_D4.0mm, F.Cu at (119.4, 86.4)
- added IC1: ArduinoProMini, mysensors_arduino:pro_mini, F.Cu at (105.4, 106.7)
- added J1: Conn_01x02_Male, Pin_Headers:Pin_Header_Straight_1x02_Pitch2.54mm, F.Cu at (92.7, 118.1)
- added J2: Conn_01x06, Pin_Headers:Pin_Header_Straight_1x06_Pitch2.54mm, F.Cu at (124.5, 99.1)
- added R1: R, Resistors_THT:R_Axial_DIN0207_L6.3mm_D2.5mm_P10.16mm_Horizontal, F.Cu at (118.1, 94.0)
- added U1: NRF24L01, mysensors_radios:NRF24L01, F.Cu at (97.8, 77.5)
Routing:
- net GND: track 0.00 -> 98.6 mm
- net /3.3V: track 0.00 -> 47.3 mm
- net /nRF_IRQ: track 0.00 -> 40.2 mm
- net /nRF_MOSI: track 0.00 -> 38.9 mm
- net /nRF_SCK: track 0.00 -> 29.5 mm
- net /nRF_MISO: track 0.00 -> 26.8 mm
- net /nRF_CE: track 0.00 -> 21.4 mm
- net /nRF_CSN: track 0.00 -> 21.3 mm
- net /Click_Amp: track 0.00 -> 15.1 mm
- net /PB_Start0: track 0.00 -> 12.6 mm
- net /PB_Start2: track 0.00 -> 12.6 mm
- net /PB_Start1: track 0.00 -> 12.6 mm
- net /PB_Start3: track 0.00 -> 12.6 mm
- net /PB_Stop: track 0.00 -> 12.0 mm
- net Net-(IC1-Pad28): track 0.00 -> 10.3 mm
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
Commit message: wip
Parts:
- added SW1: SW_Push, Buttons_Switches_THT:SW_PUSH_6mm_h8mm, F.Cu at (147.3, 116.8)
- added SW2: SW_Push, Buttons_Switches_THT:SW_PUSH_6mm_h8mm, F.Cu at (172.7, 116.8)
- added SW3: SW_Push, Buttons_Switches_THT:SW_PUSH_6mm_h8mm, F.Cu at (146.1, 88.9)
- added SW4: SW_Push, Buttons_Switches_THT:SW_PUSH_6mm_h8mm, F.Cu at (172.7, 88.9)
- added SW5: SW_Push, Buttons_Switches_THT:SW_PUSH_6mm_h8mm, F.Cu at (201.9, 88.9)
- J2: value Conn_01x06 -> Barrel_Jack; footprint Pin_Headers:Pin_Header_Straight_1x06_Pitch2.54mm -> mysensors_connectors:dc_socket-kcswalter
- moved J1 46.5 mm to (119.4, 80.0)
- moved J2 41.5 mm to (86.4, 115.6), turned to 270 degrees
- moved C1 8.89 mm to (92.7, 82.5)
- moved U1 8.89 mm to (97.8, 86.4)
Connections:
- J2 pad 1: /PB_Start3 -> +5V
- J2 pad 2: /PB_Start2 -> GND
- J2 pad 3: /PB_Start1 -> Net-(J2-Pad3)
Routing:
- net GND: track 98.6 -> 323.4 mm
- net /PB_Start3: track 12.6 -> 99.1 mm
- net /PB_Start2: track 12.6 -> 72.1 mm
- net /PB_Start0: track 12.6 -> 70.9 mm
- net /Click_Amp: track 15.1 -> 48.9 mm
- net /PB_Start1: track 12.6 -> 45.3 mm
- net /PB_Stop: track 12.0 -> 44.5 mm
- net /nRF_MOSI: track 38.9 -> 21.2 mm
- net /nRF_MISO: track 26.8 -> 17.9 mm
- net /nRF_CSN: track 21.3 -> 13.0 mm
- net /nRF_IRQ: track 40.2 -> 32.1 mm
- net +5V: track 0.00 -> 8.02 mm
- net /nRF_SCK: track 29.5 -> 21.8 mm
- net /nRF_CE: track 21.4 -> 14.8 mm
- net /3.3V: track 47.3 -> 41.6 mm
- added copper zone on B.Cu, net GND
Other:
- board outline added: 141 x 76.2 mm

Commit message: wip
Parts:
- added C2: 10nF, Capacitors_SMD:C_0603, F.Cu at (141.0, 74.9)
- added C3: 10pF, Capacitors_SMD:C_0603, F.Cu at (149.9, 64.8)
- added C4: C, Capacitors_SMD:C_0603, F.Cu at (146.1, 67.3)
- added C5: 100uF, Capacitors_THT:CP_Radial_D6.3mm_P2.50mm, F.Cu at (154.9, 67.3)
- added D2: LED, LEDs:LED_0603, F.Cu at (135.9, 67.3)
- added J3: Conn_01x04_Male, Pin_Headers:Pin_Header_Straight_1x04_Pitch2.54mm, F.Cu at (129.5, 66.0)
- added J4: Screw_Terminal_01x02, mysensors_connectors:TerminalBlock2.54mmx2-kcswalter, F.Cu at (165.1, 69.8)
- added R2: 1K, Resistors_SMD:R_0603, F.Cu at (134.6, 64.8)
- added R3: 0, Resistors_SMD:R_0603, F.Cu at (142.2, 64.8)
- added R4: 100, Resistors_SMD:R_0603, F.Cu at (139.7, 67.3)
- added RV1: 10K, Potentiometers:Potentiometer_Trimmer_ACP_CA6v_Horizontal, F.Cu at (133.3, 69.8)
- added U2: LM386, SMD_Packages:SOIC-8-N, F.Cu at (147.3, 73.7)
- J1: value Conn_01x02_Male -> Barrel_Jack; footprint Pin_Headers:Pin_Header_Straight_1x02_Pitch2.54mm -> mysensors_connectors:dc_socket-kcswalter
- J2: value Barrel_Jack -> Conn_01x02_Male; footprint mysensors_connectors:dc_socket-kcswalter -> Pin_Headers:Pin_Header_Straight_1x02_Pitch2.54mm
- R1: footprint Resistors_THT:R_Axial_DIN0207_L6.3mm_D2.5mm_P10.16mm_Horizontal -> Resistors_THT:R_Axial_DIN0204_L3.6mm_D1.6mm_P5.08mm_Horizontal
- moved J2 50.4 mm to (119.4, 77.5), turned to 180 degrees
- moved J1 48.5 mm to (86.4, 115.6), turned to 270 degrees
Connections:
- IC1 pad 1: Net-(IC1-Pad1) -> (no net)
- IC1 pad 18: Net-(IC1-Pad18) -> (no net)
- IC1 pad 19: Net-(IC1-Pad19) -> (no net)
- IC1 pad 2: Net-(IC1-Pad2) -> (no net)
- IC1 pad 20: Net-(IC1-Pad20) -> (no net)
- IC1 pad 22: Net-(IC1-Pad22) -> (no net)
- IC1 pad 25: Net-(IC1-Pad25) -> (no net)
- IC1 pad 26: Net-(IC1-Pad26) -> (no net)
- IC1 pad 3: Net-(IC1-Pad3) -> (no net)
- J1 pad 1: GND -> +5V
- J1 pad 2: /Click_Amp -> GND
- J2 pad 1: +5V -> GND
- J2 pad 2: GND -> /Click_Amp
Routing:
- net GND: track 323.4 -> 8.27 mm, vias 0 -> 5
- net +5V: track 8.02 -> 121.6 mm
- net Net-(C4-Pad1): track 0.00 -> 24.7 mm, vias 0 -> 1
- net Net-(R3-Pad2): track 0.00 -> 12.4 mm
- net Net-(C3-Pad2): track 0.00 -> 10.5 mm
- net Net-(RV1-Pad2): track 0.00 -> 10.3 mm
- net Net-(C2-Pad2): track 0.00 -> 10.0 mm
- net /Click_Amp: track 48.9 -> 58.7 mm
- net Net-(C5-Pad2): track 0.00 -> 9.24 mm
- net Net-(C4-Pad2): track 0.00 -> 8.77 mm
- net Net-(C3-Pad1): track 0.00 -> 8.11 mm
- net /3.3V: track 41.6 -> 45.4 mm
- net Net-(D2-Pad2): track 0.00 -> 3.45 mm
- net Net-(D1-Pad2): track 10.3 -> 8.15 mm
- added copper zone on F.Cu, net GND
Other:
- board size 141 x 76.2 mm -> 135.9 x 76.2 mm

Commit message: wip
Routing:
- net /PB_Start2: track 72.1 -> 75.1 mm
Changed lines of the file:
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@@
   )
   (setup
-    (last_trace_width 0.25)
+    (last_trace_width 1)
     (user_trace_width 0.25)
     (user_trace_width 0.5)
@@
   (segment (start 112.611 110.49) (end 112.467 110.634) (width 0.25) (layer F.Cu) (net 6))
   (segment (start 113.03 110.49) (end 112.611 110.49) (width 0.25) (layer F.Cu) (net 6))
-  (segment (start 139.7 109.22) (end 147.32 116.84) (width 0.25) (layer F.Cu) (net 7))
-  (segment (start 116.84 109.22) (end 139.7 109.22) (width 0.25) (layer F.Cu) (net 7))
-  (segment (start 115.57 107.95) (end 116.84 109.22) (width 0.25) (layer F.Cu) (net 7))
-  (segment (start 113.03 107.95) (end 115.57 107.95) (width 0.25) (layer F.Cu) (net 7))
+  (segment (start 139.7 109.22) (end 147.32 116.84) (width 1) (layer F.Cu) (net 7))
+  (segment (start 113.03 107.95) (end 115.57 107.95) (width 1) (layer F.Cu) (net 7))
+  (segment (start 115.57 107.95) (end 116.84 109.22) (width 1) (layer F.Cu) (net 7))
+  (segment (start 116.84 109.22) (end 139.7 109.22) (width 1) (layer F.Cu) (net 7))
   (segment (start 153.82 116.84) (end 147.32 116.84) (width 0.25) (layer F.Cu) (net 7))
-  (segment (start 162.56 106.68) (end 172.72 116.84) (width 0.25) (layer F.Cu) (net 8))
-  (segment (start 118.11 106.68) (end 162.56 106.68) (width 0.25) (layer F.Cu) (net 8))
-  (segment (start 116.84 105.41) (end 118.11 106.68) (width 0.25) (layer F.Cu) (net 8))
-  (segment (start 113.03 105.41) (end 116.84 105.41) (width 0.25) (layer F.Cu) (net 8))
+  (segment (start 162.56 106.68) (end 172.72 116.84) (width 1) (layer F.Cu) (net 8))
+  (segment (start 113.03 105.41) (end 116.84 105.41) (width 1) (layer F.Cu) (net 8))
+  (segment (start 116.84 105.41) (end 118.11 106.68) (width 1) (layer F.Cu) (net 8))
+  (segment (start 118.11 106.68) (end 162.56 106.68) (width 1) (layer F.Cu) (net 8))
   (segment (start 179.22 116.84) (end 172.72 116.84) (width 0.25) (layer F.Cu) (net 8))
   (segment (start 152.55 88.9) (end 146.05 88.9) (width 0.25) (layer F.Cu) (net 9))
-  (segment (start 132.08 102.87) (end 113.03 102.87) (width 0.25) (layer B.Cu) (net 9))
-  (segment (start 146.05 88.9) (end 132.08 102.87) (width 0.25) (layer B.Cu) (net 9))
+  (segment (start 132.08 102.87) (end 113.03 102.87) (width 1) (layer B.Cu) (net 9))
+  (segment (start 146.05 88.9) (end 132.08 102.87) (width 1) (layer B.Cu) (net 9))
   (segment (start 179.22 88.9) (end 172.72 88.9) (width 0.25) (layer F.Cu) (net 10))
-  (segment (start 124.643 100.33) (end 113.03 100.33) (width 0.25) (layer B.Cu) (net 10))
-  (segment (start 137.511 87.4622) (end 124.643 100.33) (width 0.25) (layer B.Cu) (net 10))
-  (segment (start 171.282 87.4622) (end 137.511 87.4622) (width 0.25) (layer B.Cu) (net 10))
-  (segment (start 172.72 88.9) (end 171.282 87.4622) (width 0.25) (layer B.Cu) (net 10))
+  (segment (start 124.643 100.33) (end 113.03 100.33) (width 1) (layer B.Cu) (net 10))
+  (segment (start 172.72 88.9) (end 171.282 85.5572) (width 1) (layer B.Cu) (net 10))
+  (segment (start 171.282 85.5572) (end 137.511 85.5572) (width 1) (layer B.Cu) (net 10))
+  (segment (start 137.511 85.5572) (end 124.643 100.33) (width 1) (layer B.Cu) (net 10))
   (segment (start 208.43 88.9) (end 201.93 88.9) (width 0.25) (layer F.Cu) (net 11))
-  (segment (start 128.154 97.79) (end 113.03 97.79) (width 0.25) (layer F.Cu) (net 11))
-  (segment (start 134.794 91.15) (end 128.154 97.79) (width 0.25) (layer F.Cu) (net 11))
-  (segment (start 199.68 91.15) (end 134.794 91.15) (width 0.25) (layer F.Cu) (net 11))
-  (segment (start 201.93 88.9) (end 199.68 91.15) (width 0.25) (layer F.Cu) (net 11))
+  (segment (start 128.154 97.79) (end 113.03 97.79) (width 1) (layer F.Cu) (net 11))
+  (segment (start 201.93 88.9) (end 199.68 91.15) (width 1) (layer F.Cu) (net 11))
+  (segment (start 199.68 91.15) (end 134.794 91.15) (width 1) (layer F.Cu) (net 11))
+  (segment (start 134.794 91.15) (end 128.154 97.79) (width 1) (layer F.Cu) (net 11))
   (segment (start 116.84 95.25) (end 118.11 93.98) (width 0.25) (layer F.Cu) (net 12))
   (segment (start 113.03 95.25) (end 116.84 95.25) (width 0.25) (layer F.Cu) (net 12))
@@
   (segment (start 153.67 75.565) (end 150.495 75.565) (width 1) (layer F.Cu) (net 23))
   (via (at 145.0956 69.2901) (size 0.6) (drill 0.4) (layers F.Cu B.Cu) (net 23))
-  (segment (start 147.0757 67.31) (end 145.0956 69.2901) (width 0.25) (layer B.Cu) (net 23))
-  (segment (start 154.94 67.31) (end 147.0757 67.31) (width 0.25) (layer B.Cu) (net 23))
+  (segment (start 145.0956 69.2901) (end 145.3 69.0857) (width 1) (layer F.Cu) (net 23))
   (segment (start 145.3 69.0857) (end 145.3 67.31) (width 0.25) (layer F.Cu) (net 23))
-  (segment (start 145.0956 69.2901) (end 145.3 69.0857) (width 0.25) (layer F.Cu) (net 23))
+  (segment (start 154.94 67.31) (end 147.0757 67.31) (width 1) (layer B.Cu) (net 23))
+  (segment (start 147.0757 67.31) (end 145.0956 69.2901) (width 1) (layer B.Cu) (net 23))
   (segment (start 145.9602 66.4702) (end 146.8 67.31) (width 0.25) (layer F.Cu) (net 24))
   (segment (start 140.0243 66.4702) (end 145.9602 66.4702) (width 0.25) (layer F.Cu) (net 24))
@@
     (polygon
       (pts
-        (xy 80.01 54.61) (xy 213.36 54.61) (xy 213.36 128.27) (xy 80.01 128.27)
+        (xy 213.36 128.27) (xy 80.01 128.27) (xy 80.01 54.61) (xy 213.36 54.61)
       )
     )

Commit message: wip
Parts:
- turned J4 to 90 degrees
Routing:
- net Net-(C5-Pad2): track 9.24 -> 5.39 mm
- net GND: track 8.27 -> 12.1 mm
Changed lines of the file:
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@@
   (general
     (links 65)
-    (no_connects 0)
+    (no_connects 2)
     (area 78.689999 53.289999 214.680001 129.590001)
     (thickness 1.6)
@@
   )
   (setup
-    (last_trace_width 1)
+    (last_trace_width 0.25)
     (user_trace_width 0.25)
     (user_trace_width 0.5)
@@
     (pad 29 thru_hole oval (at 13.97 0 90) (size 2.19964 1.50114) (drill 0.8001) (layers *.Cu *.Mask F.SilkS)
       (net 2 GND))
-    (model Socket_Strips.3dshapes/Socket_Strip_Straight_1x02.wrl
-      (at (xyz -0.15 0.2 0))
-      (scale (xyz 1 1 1))
-      (rotate (xyz 0 0 0))
-    )
-    (model Socket_Strips.3dshapes/Socket_Strip_Straight_1x03.wrl
-      (at (xyz 0.55 0.1 0))
-      (scale (xyz 1 1 1))
-      (rotate (xyz 0 0 90))
-    )
-    (model Socket_Strips.3dshapes/Socket_Strip_Straight_1x12.wrl
-      (at (xyz 0 0.3 0))
-      (scale (xyz 1 1 1))
-      (rotate (xyz 0 0 0))
-    )
-    (model Socket_Strips.3dshapes/Socket_Strip_Straight_1x12.wrl
-      (at (xyz 0 -0.3 0))
-      (scale (xyz 1 1 1))
-      (rotate (xyz 0 0 0))
-    )
-    (model Socket_Strips.3dshapes/Socket_Strip_Straight_1x02.wrl
-      (at (xyz 0.25 0.2 0))
-      (scale (xyz 1 1 1))
-      (rotate (xyz 0 0 0))
-    )
     (model ${MYSLOCAL}/mysensors.3dshapes/mysensors_arduino.3dshapes/arduino_pro_mini.wrl
-      (at (xyz -0.05 0 0.48))
+      (at (xyz -0.05 0 0.18))
       (scale (xyz 0.395 0.395 0.395))
       (rotate (xyz 0 0 180))
     )
     (model SMD_Packages.3dshapes/TQFP-32.wrl
-      (at (xyz 0.05 0 0.5125))
+      (at (xyz 0.05 0 0.2125))
       (scale (xyz 1 1 1))
       (rotate (xyz 0 0 315))
     )
-    (model Pin_Headers.3dshapes/Pin_Header_Straight_1x12.wrl
-      (at (xyz 0 -0.3 0.445))
-      (scale (xyz 1 1 1))
-      (rotate (xyz 0 180 0))
-    )
-    (model Pin_Headers.3dshapes/Pin_Header_Straight_1x12.wrl
-      (at (xyz 0 0.3 0.445))
-      (scale (xyz 1 1 1))
-      (rotate (xyz 0 180 0))
-    )
-    (model Pin_Headers.3dshapes/Pin_Header_Straight_1x03.wrl
-      (at (xyz 0.55 0.1 0.445))
-      (scale (xyz 1 1 1))
-      (rotate (xyz 0 180 90))
-    )
-    (model Pin_Headers.3dshapes/Pin_Header_Straight_1x02.wrl
-      (at (xyz 0.25 0.2 0.445))
-      (scale (xyz 1 1 1))
-      (rotate (xyz 0 180 0))
-    )
-    (model Pin_Headers.3dshapes/Pin_Header_Straight_1x02.wrl
-      (at (xyz -0.15 0.2 0.445))
-      (scale (xyz 1 1 1))
-      (rotate (xyz 0 180 0))
+    (model Pin_Headers.3dshapes/Pin_Header_Straight_1x12_Pitch2.54mm.wrl
+      (at (xyz -0.55 -0.3 0.145))
+      (scale (xyz 1 1 1))
+      (rotate (xyz 0 180 -90))
+    )
+    (model Pin_Headers.3dshapes/Pin_Header_Straight_1x12_Pitch2.54mm.wrl
+      (at (xyz -0.55 0.3 0.145))
+      (scale (xyz 1 1 1))
+      (rotate (xyz 0 180 -90))
     )
     (model ${MYSLOCAL}/mysensors.3dshapes/w.lain.3dshapes/smd_leds/led_0603.wrl
-      (at (xyz -0.3 0 0.5125))
+      (at (xyz -0.3 0 0.2125))
       (scale (xyz 1 1 1))
       (rotate (xyz 0 0 0))
     )
     (model ${MYSLOCAL}/mysensors.3dshapes/w.lain.3dshapes/smd_leds/led_0603.wrl
-      (at (xyz 0.55 -0.175 0.5125))
-      (scale (xyz 1 1 1))
-      (rotate (xyz 0 0 0))
-    )
-    (model Pin_Headers.3dshapes/Pin_Header_Angled_1x06.wrl
-      (at (xyz -0.65 0 0.5125))
-      (scale (xyz 1 1 1))
-      (rotate (xyz 0 0 270))
+      (at (xyz 0.55 -0.175 0.2125))
+      (scale (xyz 1 1 1))
+      (rotate (xyz 0 0 0))
     )
     (model Resistors_SMD.3dshapes/R_0603.wrl
-      (at (xyz -0.3 -0.05 0.5125))
+      (at (xyz -0.3 -0.05 0.2125))
       (scale (xyz 1 1 1))
       (rotate (xyz 0 0 0))
     )
     (model Resistors_SMD.3dshapes/R_0603.wrl
-      (at (xyz 0.55 -0.125 0.5125))
+      (at (xyz 0.55 -0.125 0.2125))
       (scale (xyz 1 1 1))
       (rotate (xyz 0 0 0))
     )
     (model Capacitors_SMD.3dshapes/C_0603.wrl
-      (at (xyz -0.3 0.05 0.5125))
+      (at (xyz -0.3 0.05 0.2125))
       (scale (xyz 1 1 1))
       (rotate (xyz 0 0 0))
     )
     (model Capacitors_Tantalum_SMD.3dshapes/TantalC_SizeS_EIA-3216.wrl
-      (at (xyz -0.35 0.15 0.5125))
+      (at (xyz -0.35 0.15 0.2125))
       (scale (xyz 1 1 1))
       (rotate (xyz 0 0 0))
     )
     (model Capacitors_Tantalum_SMD.3dshapes/TantalC_SizeS_EIA-3216.wrl
-      (at (xyz -0.35 -0.15 0.5125))
+      (at (xyz -0.35 -0.15 0.2125))
       (scale (xyz 1 1 1))
       (rotate (xyz 0 0 0))
     )
     (model TO_SOT_Packages_SMD.3dshapes/SOT-23-5.wrl
-      (at (xyz -0.4 0 0.5125))
+      (at (xyz -0.4 0 0.2125))
       (scale (xyz 1 1 1))
       (rotate (xyz 0 0 90))
     )
     (model Capacitors_SMD.3dshapes/C_1210.wrl
-      (at (xyz -0.5 0 0.5125))
+      (at (xyz -0.5 0 0.2125))
       (scale (xyz 1 1 1))
       (rotate (xyz 0 0 90))
@@
     (pad 2 thru_hole oval (at -1.524 4.064 180) (size 1.7272 1.7272) (drill 1.016) (layers *.Cu *.Mask F.SilkS)
       (net 1 /3.3V))
-    (model Socket_Strips.3dshapes/Socket_Strip_Straight_2x04.wrl
-      (at (xyz -0.21 -0.11 0))
-      (scale (xyz 1 1 1))
-      (rotate (xyz 0 0 0))
-    )
-    (model Pin_Headers.3dshapes/Pin_Header_Straight_2x04.wrl
-      (at (xyz -0.21 -0.11 0.442))
-      (scale (xyz 1 1 1))
-      (rotate (xyz 0 180 0))
+    (model Pin_Headers.3dshapes/Pin_Header_Straight_2x04_Pitch2.54mm.wrl
+      (at (xyz -0.06 -0.16 0.142))
+      (scale (xyz 1 1 1))
+      (rotate (xyz 0 180 90))
     )
     (model ${MYSLOCAL}/mysensors.3dshapes/mysensors_radios.3dshapes/nrf24l01.wrl
-      (at (xyz -0.3 -0.5669999999999999 0.475))
+      (at (xyz -0.3 -0.5669999999999999 0.175))
       (scale (xyz 0.395 0.395 0.395))
       (rotate (xyz 0 0 0))
     )
     (model Housings_DFN_QFN.3dshapes/QFN-20-1EP_4x4mm_Pitch0.5mm.wrl
-      (at (xyz -0.22 -0.51 0.509))
+      (at (xyz -0.22 -0.51 0.209))
       (scale (xyz 1 1 1))
       (rotate (xyz 0 0 0))
     )
     (model ${MYSLOCAL}/mysensors.3dshapes/w.lain.3dshapes/crystal/crystal_hc-49s.wrl
-      (at (xyz -0.5 -0.475 0.51))
+      (at (xyz -0.5 -0.475 0.21))
       (scale (xyz 1 1 1))
       (rotate (xyz 0 0 90))
@@
   )
   (module mysensors_connectors:TerminalBlock2.54mmx2-kcswalter (layer F.Cu)
-    (at 165.1 69.85 270)
+    (at 165.1 69.85 90)
     (descr "2-way 2.54mm pitch terminal block, Phoenix MPT series")
-    (fp_text reference J4 (at 0 -4.50088 270) (layer F.SilkS) hide
+    (fp_text reference J4 (at 0 -4.50088 90) (layer F.SilkS) hide
       (effects (font (thickness 0.3048)))
     )
-    (fp_text value Screw_Terminal_01x02 (at 0 4.50088 270) (layer F.SilkS) hide
+    (fp_text value Screw_Terminal_01x02 (at 0 4.50088 90) (layer F.SilkS) hide
       (effects (font (thickness 0.3048)))
     )
@@
     (fp_line (start 2.79908 -3.0988) (end -2.79908 -3.0988) (layer F.SilkS) (width 0.254))
     (fp_line (start -2.79908 -3.0988) (end -2.79908 3.0988) (layer F.SilkS) (width 0.254))
-    (pad 2 thru_hole oval (at -1.27 0 270) (size 1.99898 1.99898) (drill 1.09728) (layers *.Cu *.Mask F.SilkS)
-      (net 2 GND))
-    (pad 1 thru_hole rect (at 1.27 0 270) (size 1.99898 1.99898) (drill 1.09728) (layers *.Cu *.Mask F.SilkS)
+    (pad 2 thru_hole oval (at -1.27 0 90) (size 1.99898 1.99898) (drill 1.09728) (layers *.Cu *.Mask F.SilkS)
+      (net 2 GND))
+    (pad 1 thru_hole rect (at 1.27 0 90) (size 1.99898 1.99898) (drill 1.09728) (layers *.Cu *.Mask F.SilkS)
       (net 25 "Net-(C5-Pad2)"))
     (model ${MYSLOCAL}/mysensors.3dshapes/w.lain.3dshapes/conn_mpt/mpt_0,5-2-2,54.wrl
@@
   (segment (start 143.0757 73.1475) (end 143.1982 73.025) (width 0.25) (layer F.Cu) (net 2))
   (segment (start 141.7712 73.1475) (end 143.0757 73.1475) (width 0.25) (layer F.Cu) (net 2))
+  (segment (start 165.1 71.12) (end 161.25 71.12) (width 1) (layer B.Cu) (net 2))
   (segment (start 121.92 91.6347) (end 121.92 86.36) (width 0.25) (layer B.Cu) (net 3))
   (segment (start 123.19 92.9047) (end 121.92 91.6347) (width 0.25) (layer B.Cu) (net 3))
@@
   (segment (start 138.95 67.31) (end 139.5753 67.31) (width 0.25) (layer F.Cu) (net 24))
   (segment (start 161.25 71.12) (end 157.44 67.31) (width 1) (layer B.Cu) (net 25))
-  (segment (start 165.1 71.12) (end 161.25 71.12) (width 1) (layer B.Cu) (net 25))
   (segment (start 135.9953 65.84) (end 136.69 66.5347) (width 0.25) (layer F.Cu) (net 26))
   (segment (start 135.9953 64.77) (end 135.9953 65.84) (width 0.25) (layer F.Cu) (net 26))
